File: kicad/pcb/pcb.kicad_pcb (KiCad board)
At the start: 2 copper layers, 303.7 x 99.9 mm, 123 parts, among them SW1 RotaryEncoder_Switch, U1 Teensy2.0_(Arduino)

Commit message: edits before formatting mac
Parts:
- removed G***: LOGO, LOGO
- removed LED0: Conn_01x03_Female, Connector_PinHeader_2.54mm:PinHeader_1x03_P2.54mm_Vertical
- removed OLED0: Conn_01x04_Female, Connector_PinHeader_2.54mm:PinHeader_1x04_P2.54mm_Vertical
- added LED1: Conn_01x03_Female, Connector_PinHeader_2.54mm:PinHeader_1x03_P2.54mm_Vertical, F.Cu at (64.0, 149.7)
- added OLED1: Conn_01x04_Female, Connector_PinHeader_2.54mm:PinHeader_1x04_P2.54mm_Vertical, F.Cu at (59.4, 149.7)
- D10, D11, D12, D13, D14, D15, D16, D17, D18, D19, D2, D20, D21, D22, D23, D24, D25, D26, D27, D28, D29, D3, D30, D31, D32, D33, D34, D35, D36, D37, D38, D39, D4, D40, D41, D42, D43, D44, D45, D46, D47, D48, D49, D5, D50, D51, D52, D53, D54, D6, D7, D8, D9: moved to F.Cu
- moved D27 306.9 mm to (48.0, 163.2), turned to 0 degrees
- moved D28 282.8 mm to (92.5, 162.0), turned to 0 degrees
- moved D13 275.8 mm to (82.2, 152.2), turned to 0 degrees
- moved D41 265.7 mm to (86.2, 158.8), turned to 0 degrees
- moved MX13 265.6 mm to (68.8, 96.9)
- moved MX41 263.2 mm to (68.8, 56.5)
- moved D42 260.9 mm to (111.5, 162.0), turned to 0 degrees
- moved D53 253.9 mm to (98.8, 158.8), turned to 0 degrees
- moved MX42 251.1 mm to (109.2, 137.3)
- moved D14 242.5 mm to (136.9, 149.0), turned to 0 degrees
- moved MX12 239.4 mm to (68.8, 76.7), turned to 0 degrees
- moved D10 233.0 mm to (73.5, 162.0), turned to 0 degrees
- moved D26 232.1 mm to (105.2, 155.5), turned to 0 degrees
- moved D11 229.0 mm to (98.8, 162.0), turned to 0 degrees
- moved MX26 228.2 mm to (89.0, 117.1), turned to 0 degrees
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Connections:
- D51 pad 2: Net-(D51-Pad2) -> Net-(D51-A)
- D52 pad 2: Net-(D52-Pad2) -> Net-(D52-A)
- D53 pad 2: Net-(D53-Pad2) -> Net-(D53-A)
- D54 pad 2: Net-(D54-Pad2) -> Net-(D54-A)
- MX51 pad 2: Net-(D51-Pad2) -> Net-(D52-A)
- MX52 pad 2: Net-(D52-Pad2) -> Net-(D53-A)
- MX53 pad 2: Net-(D53-Pad2) -> Net-(D54-A)
- SW1 pad S2: Net-(D54-Pad2) -> Net-(D51-A)
- U1 pad 1: unconnected-(U1-Pad1) -> GND
Routing:
- net ROW3: track 369.6 -> 0.00 mm, vias 2 -> 0
- net ROW2: track 344.3 -> 0.00 mm
- net ROW0: track 334.3 -> 0.00 mm, vias 2 -> 0
- net ROW1: track 324.5 -> 0.00 mm, vias 2 -> 0
- net COL13: track 244.5 -> 0.00 mm, vias 4 -> 0
- net COL12: track 203.7 -> 0.00 mm, vias 4 -> 0
- net COL11: track 199.3 -> 0.00 mm, vias 4 -> 0
- net COL0: track 193.2 -> 0.00 mm, vias 4 -> 0
- net COL10: track 177.1 -> 0.00 mm, vias 4 -> 0
- net COL2: track 168.1 -> 0.00 mm, vias 4 -> 0
- net COL1: track 158.3 -> 0.00 mm, vias 3 -> 0
- net COL3: track 152.5 -> 0.00 mm, vias 4 -> 0
- net COL9: track 152.2 -> 0.00 mm, vias 3 -> 0
- net COL4: track 147.3 -> 0.00 mm, vias 5 -> 0
- net COL5: track 125.0 -> 0.00 mm, vias 5 -> 0
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- removed copper zone on B.Cu, net GND
- removed copper zone on F.Cu, net GND
Other:
- board outline removed
- board text removed: "128X32 OLED MODULE"
- board text removed: "AVANTE53"
- board text removed: "Avante53 PCB Rev.2 by Pimentoso https://github.com/Pimentoso/avante53"
- board text removed: "SDA SCL VCC GND"
- board text removed: "Teensy2.0"
- board text removed: "VCC DIN GND"
- board text removed: "WS8212b LED STRIP"
