File: kicad/pcb/pcb.kicad_sch (KiCad schematic)
At the start: 122 parts, among them SW1 RotaryEncoder_Switch, U1 Teensy2.0_(Arduino)

Commit message: edits before formatting mac
Parts:
- renumbered D54 to D51, D51 to D52, D52 to D53, D53 to D54, LED0 to LED1, OLED0 to OLED1
Changed lines of the file:
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@@
   (symbol (lib_id "Connector:Conn_01x03_Female") (at 210.82 57.15 0) (unit 1)
     (in_bom yes) (on_board yes) (fields_autoplaced)
-    (property "Reference" "LED0" (id 0) (at 212.09 55.8799 0)
+    (property "Reference" "LED1" (id 0) (at 212.09 55.8799 0)
       (effects (font (size 1.27 1.27)) (justify left))
     )
@@
   (symbol (lib_id "Device:D_Small") (at 218.44 160.02 90) (unit 1)
     (in_bom yes) (on_board yes) (fields_autoplaced)
-    (property "Reference" "D52" (id 0) (at 220.98 158.7499 90)
+    (property "Reference" "D53" (id 0) (at 220.98 158.7499 90)
       (effects (font (size 1.27 1.27)) (justify right))
     )
@@
   (symbol (lib_id "Device:D_Small") (at 200.66 148.59 90) (unit 1)
     (in_bom yes) (on_board yes)
-    (property "Reference" "D54" (id 0) (at 203.2 147.3199 90)
+    (property "Reference" "D51" (id 0) (at 203.2 147.3199 90)
       (effects (font (size 1.27 1.27)) (justify right))
     )
@@
   (symbol (lib_id "Connector:Conn_01x04_Female") (at 210.82 41.91 0) (unit 1)
     (in_bom yes) (on_board yes) (fields_autoplaced)
-    (property "Reference" "OLED0" (id 0) (at 212.09 41.9099 0)
+    (property "Reference" "OLED1" (id 0) (at 212.09 41.9099 0)
       (effects (font (size 1.27 1.27)) (justify left))
     )
@@
   (symbol (lib_id "Device:D_Small") (at 207.01 160.02 90) (unit 1)
     (in_bom yes) (on_board yes) (fields_autoplaced)
-    (property "Reference" "D51" (id 0) (at 209.55 158.7499 90)
+    (property "Reference" "D52" (id 0) (at 209.55 158.7499 90)
       (effects (font (size 1.27 1.27)) (justify right))
     )
@@
   (symbol (lib_id "Device:D_Small") (at 229.87 160.02 90) (unit 1)
     (in_bom yes) (on_board yes) (fields_autoplaced)
-    (property "Reference" "D53" (id 0) (at 232.41 158.7499 90)
+    (property "Reference" "D54" (id 0) (at 232.41 158.7499 90)
       (effects (font (size 1.27 1.27)) (justify right))
     )
@@
       (reference "D50") (unit 1) (value "D_Small") (footprint "Diode_SMD:D_MiniMELF")
     )
+    (path "/52c0ce29-8b1e-4757-ac6a-784d81e8e050"
+      (reference "D51") (unit 1) (value "D_Small") (footprint "Diode_SMD:D_MiniMELF")
+    )
     (path "/cacdb716-a488-4397-8a22-585cc9ed135e"
-      (reference "D51") (unit 1) (value "D_Small") (footprint "Diode_SMD:D_MiniMELF")
+      (reference "D52") (unit 1) (value "D_Small") (footprint "Diode_SMD:D_MiniMELF")
     )
     (path "/48d1c137-5b33-4241-86cb-5aa0949a5598"
-      (reference "D52") (unit 1) (value "D_Small") (footprint "Diode_SMD:D_MiniMELF")
+      (reference "D53") (unit 1) (value "D_Small") (footprint "Diode_SMD:D_MiniMELF")
     )
     (path "/d9daafa3-61cd-4d0a-aa94-c29e67b1a7a7"
-      (reference "D53") (unit 1) (value "D_Small") (footprint "Diode_SMD:D_MiniMELF")
-    )
-    (path "/52c0ce29-8b1e-4757-ac6a-784d81e8e050"
       (reference "D54") (unit 1) (value "D_Small") (footprint "Diode_SMD:D_MiniMELF")
     )
@@
     )
     (path "/267d0249-a9ed-4c0d-987b-0e9e8385f620"
-      (reference "LED0") (unit 1) (value "Conn_01x03_Female") (footprint "Connector_PinHeader_2.54mm:PinHeader_1x03_P2.54mm_Vertical")
+      (reference "LED1") (unit 1) (value "Conn_01x03_Female") (footprint "Connector_PinHeader_2.54mm:PinHeader_1x03_P2.54mm_Vertical")
     )
     (path "/7256b151-a8ca-4762-8118-1528709e7f97"
@@
     )
     (path "/64f53ab3-14ea-4cbd-abe9-5b7f9991e2f9"
-      (reference "OLED0") (unit 1) (value "Conn_01x04_Female") (footprint "Connector_PinHeader_2.54mm:PinHeader_1x04_P2.54mm_Vertical")
+      (reference "OLED1") (unit 1) (value "Conn_01x04_Female") (footprint "Connector_PinHeader_2.54mm:PinHeader_1x04_P2.54mm_Vertical")
     )
     (path "/c266ebe0-572c-41c9-9c58-4ebe1191562c"
